File: BigProject2/PCB_ADC/pcd_adc.kicad_pcb (KiCad board)
At the start: 2 copper layers, 28 parts, among them J1 I2C_input, J2 I2C_input, SW1 Mode_Calib, U1 ATmega328P-P, U2 LCD-16X2, Y1 16MHz

Commit message: up
Parts:
- U1: moved to B.Cu
- moved BTN1 278.1 mm to (187.8, 86.0), turned to -90 degrees
- moved Y1 270.2 mm to (155.7, 84.3), turned to 0 degrees
- moved BTN2 227.4 mm to (132.4, 91.5)
- moved U2 78.5 mm to (170.5, 68.5)
- moved U1 53.9 mm to (179.2, 76.0), turned to 90 degrees
- moved VR1 49.2 mm to (14.6, 43.0)
Routing:
- net /PC2: track 60.1 -> 0.00 mm
- net /PC1: track 56.6 -> 0.00 mm
- net /PC0: track 53.0 -> 0.00 mm
- net /PB2: track 41.7 -> 0.00 mm
- net /PB3: track 38.0 -> 0.00 mm
- net /PB5: track 30.6 -> 0.00 mm
- net GND: track 21.5 -> 0.00 mm
- net /LCD_VO: track 7.82 -> 0.00 mm
- net /PB4: track 34.5 -> 27.2 mm
- net +5V: track 5.28 -> 0.00 mm
Other:
- board outline added: 80 x 50 mm

Commit message: up
Parts:
- removed BTN3: RESET, Button_Switch_THT:SW_PUSH_6mm
- removed C4: 100nF, Capacitor_SMD:C_1206_3216Metric
- removed C7: 100nF, Capacitor_THT:C_Disc_D7.5mm_W5.0mm_P7.50mm
- removed L1: 10uH, Inductor_SMD:L_1210_3225Metric
- C5: footprint Capacitor_SMD:C_1206_3216Metric -> Capacitor_THT:C_Disc_D7.5mm_W5.0mm_P7.50mm; moved to F.Cu
- R8: footprint Resistor_THT:R_Axial_DIN0207_L6.3mm_D2.5mm_P10.16mm_Horizontal -> Resistor_SMD:R_1206_3216Metric; moved to B.Cu
- moved C6 373.8 mm to (199.0, 64.2), turned to -90 degrees
- moved R7 362.0 mm to (202.4, 78.2), turned to 180 degrees
- moved C8 357.6 mm to (188.0, 99.0), turned to 90 degrees
- moved R5 353.9 mm to (202.4, 81.3), turned to 180 degrees
- moved R4 350.1 mm to (202.4, 84.4), turned to 180 degrees
- moved R8 349.2 mm to (174.0, 57.5), turned to 90 degrees
- moved C9 346.6 mm to (175.0, 99.0), turned to 90 degrees
- moved R6 330.2 mm to (172.8, 79.4), turned to 180 degrees
- moved C1 305.4 mm to (175.6, 77.0)
- moved R2 296.2 mm to (149.7, 75.0), turned to 180 degrees
- moved C2 295.7 mm to (170.0, 77.1)
- moved R3 285.2 mm to (139.9, 91.5)
- moved SW1 261.7 mm to (205.0, 67.5), turned to -90 degrees
- moved C3 252.8 mm to (177.0, 57.5), turned to -90 degrees
- moved R1 216.8 mm to (149.7, 71.2), turned to 180 degrees
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Connections:
- U1 pad 20: Net-(U1-AVCC) -> +5V
- U2 pad 7: unconnected-(U2-DB0-Pad7) -> GND
Routing:
- net GND: track 0.00 -> 415.2 mm, vias 0 -> 4
- net +5V: track 0.00 -> 174.8 mm
- net /SCL: track 0.00 -> 82.6 mm, vias 0 -> 2
- net /SDA: track 0.00 -> 73.2 mm, vias 0 -> 2
- net /PC2: track 0.00 -> 59.9 mm
- net /PC1: track 0.00 -> 52.6 mm
- net /PD3: track 0.00 -> 52.0 mm
- net /PD2: track 0.00 -> 47.0 mm
- net /PC0: track 0.00 -> 44.8 mm
- net /PD0: track 0.00 -> 32.0 mm
- net /LCD_VO: track 0.00 -> 29.0 mm
- net /PB4: track 27.2 -> 9.88 mm
- net Net-(U1-XTAL1/PB6): track 0.00 -> 11.1 mm
- net Net-(U1-XTAL2/PB7): track 0.00 -> 11.1 mm
- net /PB5: track 0.00 -> 9.91 mm
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- added copper zone on B.Cu, net GND
Other:
- board size 80 x 50 mm -> 100.5 x 70 mm

Commit message: up date PCB
Parts:
- moved VR1 5.26 mm to (139.2, 59.0)
- moved I2C_input 1.17 mm to (133.7, 74.5)
- renumbered SW1 to CALIB_MODE, J1 to I2C_input, J2 to POWER_CONN, BTN2 to SAVE_MODE, BTN1 to SELECT_MODE
Routing:
- net GND: track 415.2 -> 368.3 mm
- net +5V: track 174.8 -> 185.3 mm, vias 0 -> 3
- net /LCD_VO: track 29.0 -> 19.4 mm
- net /PD0: track 32.0 -> 36.4 mm
- net /SDA: track 73.2 -> 69.0 mm, vias 2 -> 1
- net /SCL: track 82.6 -> 80.5 mm, vias 2 -> 1

Commit message: up code
Parts:
- added D1: LED, LED_SMD:LED_0805_2012Metric, B.Cu at (153.4, 84.8)
- added D2: LED, LED_SMD:LED_0805_2012Metric, B.Cu at (160.7, 84.8)
- added D3: LED, LED_SMD:LED_0805_2012Metric, B.Cu at (156.9, 84.8)
- added R10: 10k, Resistor_SMD:R_1206_3216Metric, B.Cu at (160.7, 79.3)
- added R11: 10k, Resistor_SMD:R_1206_3216Metric, B.Cu at (156.9, 79.3)
- added R9: 10k, Resistor_SMD:R_1206_3216Metric, B.Cu at (153.4, 79.3)
- moved C5 0.10 mm to (147.4, 97.5)
- renumbered SELECT_MODE to BTN1, SAVE_MODE to BTN2, I2C_input to J1, POWER_CONN to J2, CALIB_MODE to SW1
Connections:
- U1 pad 12: unconnected-(U1-PD6-Pad12) -> /PD6
- U1 pad 13: unconnected-(U1-PD7-Pad13) -> /PD7
- U1 pad 14: unconnected-(U1-PB0-Pad14) -> /PB0
Routing:
- net GND: track 368.3 -> 530.2 mm
- net /PB0: track 0.00 -> 12.2 mm
- net /PD7: track 0.00 -> 11.5 mm
- net /PD6: track 0.00 -> 9.21 mm
- net /LCD_VO: track 19.4 -> 12.8 mm
- net Net-(D2-K): track 0.00 -> 3.09 mm
- net Net-(D1-K): track 0.00 -> 3.09 mm
- net Net-(D3-K): track 0.00 -> 3.05 mm
- net /PD0: track 36.4 -> 39.3 mm
- net /PD2: track 47.0 -> 48.8 mm
- net +5V: track 185.3 -> 183.7 mm
- net /PC2: track 59.9 -> 59.2 mm
- net /PC1: track 52.6 -> 52.0 mm
Other:
- board text added: "Noname-29-lnin"

Commit message: up docs bigproject2
Routing:
- net /SCL: track 80.3 -> 87.2 mm
- net /SDA: track 69.0 -> 75.5 mm
Changed lines of the file:
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@@
 	)
 	(segment
-		(start 191.8 58.8)
+		(start 190.45 60.15)
 		(end 177.101 73.499)
 		(width 1)
@@
 		(net 9)
 	)
+	(segment
+		(start 190.45 55.55)
+		(end 190.45 60.15)
+		(width 1)
+		(layer "F.Cu")
+		(net 9)
+	)
 	(via
-		(at 191.8 58.8)
+		(at 190.45 55.55)
 		(size 0.6)
 		(drill 0.3)
@@
 	(segment
 		(start 191.86 58.86)
-		(end 191.8 58.8)
-		(width 1)
-		(layer "B.Cu")
-		(net 9)
-	)
-	(segment
-		(start 191.86 62.69)
+		(end 191.86 62.69)
+		(width 1)
+		(layer "B.Cu")
+		(net 9)
+	)
+	(segment
+		(start 190.45 57.45)
 		(end 191.86 58.86)
 		(width 1)
+		(layer "B.Cu")
+		(net 9)
+	)
+	(segment
+		(start 190.45 55.55)
+		(end 190.45 57.45)
+		(width 1.5)
 		(layer "B.Cu")
 		(net 9)
@@
 	)
 	(segment
+		(start 139.5 71.25)
+		(end 137.499 73.251)
+		(width 1.27)
+		(layer "F.Cu")
+		(net 10)
+	)
+	(segment
+		(start 192.65 60.55)
+		(end 192.65 57.1)
+		(width 1.27)
+		(layer "F.Cu")
+		(net 10)
+	)
+	(segment
 		(start 138.671158 77.001)
 		(end 176.199 77.001)
@@
 	)
 	(segment
-		(start 139.5 71.25)
-		(end 137.499 73.251)
+		(start 176.199 77.001)
+		(end 192.65 60.55)
+		(width 1.27)
+		(layer "F.Cu")
+		(net 10)
+	)
+	(segment
+		(start 192.65 57.1)
+		(end 194.4 55.35)
 		(width 1.27)
 		(layer "F.Cu")
@@
 		(net 10)
 	)
-	(segment
-		(start 176.199 77.001)
-		(end 194.4 58.8)
-		(width 1.27)
-		(layer "F.Cu")
-		(net 10)
-	)
 	(via
-		(at 194.4 58.8)
+		(at 194.4 55.35)
 		(size 0.6)
 		(drill 0.3)
@@
 	)
 	(segment
+		(start 194.4 62.69)
+		(end 194.4 57.85)
+		(width 1)
+		(layer "B.Cu")
+		(net 10)
+	)
+	(segment
 		(start 139.5 71.25)
 		(end 138.85 71.9)
@@
 	)
 	(segment
-		(start 194.4 62.69)
-		(end 194.4 58.8)
-		(width 1)
-		(layer "B.Cu")
-		(net 10)
-	)
-	(segment
 		(start 137.1 71.9)
 		(end 137.09 71.91)
@@
 		(end 137.1 71.9)
 		(width 1.27)
+		(layer "B.Cu")
+		(net 10)
+	)
+	(segment
+		(start 194.4 57.85)
+		(end 194.4 55.35)
+		(width 1.5)
 		(layer "B.Cu")
 		(net 10)
@@
 	)
 	(zone
+		(net 0)
+		(net_name "")
+		(layer "B.Cu")
+		(hatch edge 0.5)
+		(connect_pads
+			(clearance 0)
+		)
+		(min_thickness 0.25)
+		(filled_areas_thickness no)
+		(keepout
+			(tracks allowed)
+			(vias allowed)
+			(pads allowed)
+			(copperpour not_allowed)
+			(footprints allowed)
+		)
+		(placement
+			(enabled no)
+			(sheetname "/")
+		)
+		(fill
+			(thermal_gap 0.5)
+			(thermal_bridge_width 0.5)
+		)
+		(polygon
+			(pts
+				(xy 188.25 50.55) (xy 197.15 50.55) (xy 197.15 60.55) (xy 187.15 60.45)
+			)
+		)
+	)
+	(zone

Commit message: up adc_pcb
Parts:
- moved C1 9.03 mm to (175.3, 86.0), turned to -90 degrees
- moved C2 9.01 mm to (170.5, 86.0), turned to 90 degrees
- moved R6 2.44 mm to (172.8, 77.0)
- moved Y1 2.10 mm to (170.3, 81.2)
Routing:
- net GND: track 530.2 -> 524.8 mm
- net Net-(U1-XTAL2/PB7): track 11.1 -> 12.4 mm
- net Net-(U1-XTAL1/PB6): track 11.1 -> 12.4 mm
